File: VVDAP.kicad_pcb (KiCad board)
At the start: 2 copper layers, 30 x 41.5 mm, 58 parts, among them J1 FTSH-105-01-L-DV-K, J2 USB_C_Receptacle_USB2.0_16P, J3 Conn_01x04_MountingPin, J5 Conn_ARM_SWD_TagConnect_TC203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, SW1 SW_Push, SW2 SW_Push, U1 CH32V203F6P6, U10 SN74LVC1G66DBVR, U11 MIE1W0505, U12 ADuM162N1BRZ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

Commit message: Update screw pads
Other:
- board text added: "R1.3"
- board text added: "R1.3 20260106"
- board text removed: "R1.2"
- board text removed: "R1.2 20260106"
